File: kinen_MB.sch (KiCad schematic (older format))
At the start: 3 parts, among them P1 CONN_7X2, P2 CONN_13X2

Commit message: Added feature list for KinenMFB
Parts:
- added P3: SMART2, Header_F_7x2, symbol CONN_7X2
- added P4: DUMB2, Header_F_13x2, symbol CONN_13X2
- added P5: SMART3, Header_F_7x2, symbol CONN_7X2
- added P6: DUMB3, Header_F_13x2, symbol CONN_13X2
- added P7: SMART4, Header_F_7x2, symbol CONN_7X2
- added P8: DUMB4, Header_F_13x2, symbol CONN_13X2
- P1: value CONN_7X2 -> SMART1; footprint (none) -> Header_F_7x2
- P2: value CONN_13X2 -> DUMB1; footprint (none) -> Header_F_13x2
- PCB1: footprint (none) -> PCB
Connections:
- no-connect marks 40 -> 160
Other:
- note added: "FEATURES REQUIRED\n+ Controller : Atmel SAM3X8E ARM Cortex-M3 as in Arduino Due. Runs on 3V3 ONLY :http://arduino.cc/en/Main/ArduinoBoardDue\n+ RTC with DS3231\n+ uSD Card\n+ Standard headers for FTDI, ISP, I2C/C3SB\n+ Selectable ARef - 5V0 or 3V3\n+ Raspberry-Pi interface with level translator. Allow access to all Ras-Pi GPIO pins.Xlator not reqd if system is 3V3.\n+ microUSB socket for Data (us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"
- moved on the sheet: P1, P2, PCB1
